File: builds/2.0/usbcounter/usbcounter.kicad_sch (KiCad schematic)
At the start: 49 parts, among them IC1 ATTINY826-XUR, J1 UJ2-MIBH-G-SMT-TR, J2 SMA, J3 Conn_Prog, J4 Conn_Disp, Q1 MMBT2222A, U1 FT230XS, U2 SN74LVC1Gxx, U3 MCP23008-xSO, U4 74LV8154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

Commit message: 3.0: new board
Parts:
- R1: footprint Resistor_SMD:R_0805_2012Metric_Pad1.20x1.40mm_HandSolder -> Resistor_THT:R_Axial_DIN0207_L6.3mm_D2.5mm_P10.16mm_Horizontal
Changed lines of the file:
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@@
     (property "Reference" "R1" (id 0) (at 35.56 127.635 0))
     (property "Value" "50" (id 1) (at 35.56 129.54 0))
-    (property "Footprint" "Resistor_SMD:R_0805_2012Metric_Pad1.20x1.40mm_HandSolder" (id 2) (at 34.798 128.27 90)
+    (property "Footprint" "Resistor_THT:R_Axial_DIN0207_L6.3mm_D2.5mm_P10.16mm_Horizontal" (id 2) (at 34.798 128.27 90)
       (effects (font (size 1.27 1.27)) hide)
     )
@@
     )
     (path "/e192ab3c-af17-4fd1-8347-4938804d358d"
-      (reference "R1") (unit 1) (value "50") (footprint "Resistor_SMD:R_0805_2012Metric_Pad1.20x1.40mm_HandSolder")
+      (reference "R1") (unit 1) (value "50") (footprint "Resistor_THT:R_Axial_DIN0207_L6.3mm_D2.5mm_P10.16mm_Horizontal")
     )
     (path "/5dd5aa12-5573-447f-9aa7-a63ab5147207"
