File: builds/2.2/kicad/usbcounter.kicad_pcb (KiCad board)
At the start: 2 copper layers, 91.4 x 61 mm, 50 parts, among them J1 UJ2-MIBH-G-SMT-TR, J2 RF_IN, J3 PROG, J4 DISPLAY, SW1 RESET, U1 NCP1117, U2 74LVC1G14, U3 FT231XS, U4 74LV8154, U5 AVR64DD32 TQFP32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

Commit message: 2.2 PCB: complete
Parts:
- J4: footprint Connector_PinHeader_2.54mm:PinHeader_1x04_P2.54mm_Vertical -> Connector_PinHeader_2.54mm:PinHeader_1x05_P2.54mm_Vertical
- SW1: value RESET -> SW_Push
- moved D4 32.3 mm to (65.5, 56.4), turned to 180 degrees
- moved U4 30.8 mm to (88.6, 97.0)
- moved R11 29.6 mm to (123.2, 81.3)
- moved R7 26.8 mm to (65.5, 60.2)
- moved D7 26.1 mm to (119.1, 81.3)
- moved D3 25.9 mm to (67.6, 105.2)
- moved TP3 23.7 mm to (79.2, 105.2)
- moved TP2 23.5 mm to (75.7, 105.2)
- moved R12 18.4 mm to (112.3, 60.5)
- moved R8 17.6 mm to (71.6, 105.2)
- moved C7 16.7 mm to (89.4, 88.9), turned to 90 degrees
- moved D5 16.2 mm to (84.8, 56.4), turned to 180 degrees
- moved R10 14.8 mm to (90.4, 60.2)
- moved C6 13.1 mm to (77.0, 55.9), turned to 90 degrees
- moved D2 12.6 mm to (72.4, 93.7), turned to -90 degrees
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Connections:
- J3 pad 1: VCC -> GND
- J3 pad 2: GND -> VCC
- SW1 pad 2: RESET -> GND
Routing:
- net VCC: track 0.00 -> 247.0 mm, vias 0 -> 2
- net GATE: track 0.00 -> 58.1 mm, vias 0 -> 2
- net R3: track 0.00 -> 51.3 mm
- net R2: track 0.00 -> 50.0 mm
- net R1: track 0.00 -> 48.8 mm
- net R0: track 0.00 -> 48.1 mm
- net PCRX: track 0.00 -> 46.3 mm, vias 0 -> 2
- net Y7: track 0.00 -> 45.8 mm, vias 0 -> 2
- net Y4: track 0.00 -> 45.0 mm, vias 0 -> 2
- net Y6: track 0.00 -> 43.2 mm, vias 0 -> 2
- net Y5: track 0.00 -> 43.1 mm, vias 0 -> 2
- net DISP_CLK: track 0.00 -> 43.0 mm, vias 0 -> 2
- net DISP_CS: track 0.00 -> 43.0 mm, vias 0 -> 2
- net GND: track 0.00 -> 39.0 mm, vias 0 -> 24
- net PCTX: track 0.00 -> 37.7 mm, vias 0 -> 2
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- added copper zone on B.Cu, net GND
- added copper zone on F.Cu, net GND
Other:
- board text added: "@swharden"
- board text added: "CLK"
- board text added: "COUNTING"
- board text added: "CS"
- board text added: "DATA"
- board text added: "DC"
- board text added: "DISPLAY"
- board text added: "GND"
- board text added: "INPUT"
- board text added: "LOAD"
- board text added: "POWER"
- board text added: "PROG"
- board text added: "RESET"
- board text added: "RX"
- board text added: "STATUS"
- board text added: "TX"
- board text added: "UPDI"
- board text added: "USB Counter"
- board text added: "VCC"
- board text added: "v2.2"
