File: builds/2.2/kicad/usbcounter.kicad_sch (KiCad schematic)
At the start: 50 parts, among them J1 UJ2-MIBH-G-SMT-TR, J2 RF_IN, J3 PROG, J4 DISPLAY, SW1 RESET, U1 NCP1117, U2 74LVC1G14, U3 FT231XS, U4 74LV8154, U5 AVR64DD32 TQFP32, X1 TCXO

Commit message: 2.2 PCB: complete
Parts:
- removed SW1: RESET, Button_Switch_SMD:SW_SPST_TL3342, symbol Switch:SW_MEC_5G
- added SW1: SW_Push, Button_Switch_SMD:SW_SPST_TL3342, symbol Switch:SW_Push
- J4: footprint Connector_PinHeader_2.54mm:PinHeader_1x04_P2.54mm_Vertical -> Connector_PinHeader_2.54mm:PinHeader_1x05_P2.54mm_Vertical
Connections:
- net GND: now also J3.1 (Pin_1), SW1.2; no longer J3.2 (Pin_2)
- net RESET: now also SW1.1
- net VCC: now also J3.2 (Pin_2); no longer J3.1 (Pin_1)
Other:
- moved on the sheet: C1
Changed lines of the file:
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@@
-    (stroke (width 0) (type default) (color 0 0 0 0))
-  )
-  (wire (pts (xy 212.09 125.73) (xy 205.74 125.73))
     (stroke (width 0) (type default) (color 0 0 0 0))
   )
@@
     (stroke (width 0) (type default) (color 0 0 0 0))
   )
-  (wire (pts (xy 212.09 123.19) (xy 205.74 123.19))
-    (stroke (width 0) (type default) (color 0 0 0 0))
-  )
   (polyline (pts (xy 274.32 147.32) (xy 177.8 147.32))
     (stroke (width 0) (type default) (color 0 0 0 0))
@@
     (stroke (width 0) (type default) (color 0 0 0 0))
   )
-  (wire (pts (xy 205.74 128.27) (xy 205.74 130.81))
-    (stroke (width 0) (type default) (color 0 0 0 0))
-  )
   (polyline (pts (xy 144.78 25.4) (xy 144.78 25.4))
     (stroke (width 0) (type default) (color 0 0 0 0))
@@
     (stroke (width 0) (type default) (color 0 0 0 0))
   )
-  (wire (pts (xy 252.73 125.73) (xy 252.73 127))
+  (wire (pts (xy 252.73 125.73) (xy 252.73 127.635))
     (stroke (width 0) (type default) (color 0 0 0 0))
   )
@@
   )
   (polyline (pts (xy 25.4 25.4) (xy 25.4 109.22))
-    (stroke (width 0) (type default) (color 0 0 0 0))
-  )
-  (wire (pts (xy 205.74 130.81) (xy 207.01 130.81))
     (stroke (width 0) (type default) (color 0 0 0 0))
   )
@@
     )
   )
-  (global_label "UPDI" (shape input) (at 207.01 130.81 0) (fields_autoplaced)
-    (effects (font (size 1.27 1.27)) (justify left))
-    (property "Intersheet References" "${INTERSHEET_REFS}" (id 0) (at 213.8983 130.7306 0)
+  (global_label "UPDI" (shape input) (at 205.74 128.27 0) (fields_autoplaced)
+    (effects (font (size 1.27 1.27)) (justify left))
+    (property "Intersheet References" "${INTERSHEET_REFS}" (id 0) (at 212.6283 128.1906 0)
       (effects (font (size 1.27 1.27)) (justify left) hide)
     )
@@
     (pin "2")
   )
-  (symbol (lib_id "power:GND") (at 212.09 125.73 0) (unit 1)
-    (in_bom yes) (on_board yes)
-    (property "Reference" "#PWR029" (id 0) (at 212.09 132.08 0)
-      (effects (font (size 1.27 1.27)) hide)
-    )
-    (property "Value" "GND" (id 1) (at 215.9 127 0))
-    (property "Footprint" "" (id 2) (at 212.09 125.73 0)
-      (effects (font (size 1.27 1.27)) hide)
-    )
-    (property "Datasheet" "" (id 3) (at 212.09 125.73 0)
+  (symbol (lib_id "power:GND") (at 205.74 123.19 90) (unit 1)
+    (in_bom yes) (on_board yes)
+    (property "Reference" "#PWR028" (id 0) (at 212.09 123.19 0)
+      (effects (font (size 1.27 1.27)) hide)
+    )
+    (property "Value" "GND" (id 1) (at 210.82 123.19 90))
+    (property "Footprint" "" (id 2) (at 205.74 123.19 0)
+      (effects (font (size 1.27 1.27)) hide)
+    )
+    (property "Datasheet" "" (id 3) (at 205.74 123.19 0)
       (effects (font (size 1.27 1.27)) hide)
     )
@@
     )
   )
-  (symbol (lib_id "power:VCC") (at 212.09 123.19 0) (unit 1)
-    (in_bom yes) (on_board yes)
-    (property "Reference" "#PWR028" (id 0) (at 212.09 127 0)
-      (effects (font (size 1.27 1.27)) hide)
-    )
-    (property "Value" "VCC" (id 1) (at 215.9 121.92 0))
-    (property "Footprint" "" (id 2) (at 212.09 123.19 0)
-      (effects (font (size 1.27 1.27)) hide)
-    )
-    (property "Datasheet" "" (id 3) (at 212.09 123.19 0)
+  (symbol (lib_id "power:VCC") (at 205.74 125.73 270) (unit 1)
+    (in_bom yes) (on_board yes)
+    (property "Reference" "#PWR029" (id 0) (at 201.93 125.73 0)
+      (effects (font (size 1.27 1.27)) hide)
+    )
+    (property "Value" "VCC" (id 1) (at 210.185 125.73 90))
+    (property "Footprint" "" (id 2) (at 205.74 125.73 0)
+      (effects (font (size 1.27 1.27)) hide)
+    )
+    (property "Datasheet" "" (id 3) (at 205.74 125.73 0)
       (effects (font (size 1.27 1.27)) hide)
     )
@@
     (property "Reference" "J4" (id 0) (at 227.33 116.205 0))
     (property "Value" "DISPLAY" (id 1) (at 229.87 118.11 0))
-    (property "Footprint" "Connector_PinHeader_2.54mm:PinHeader_1x04_P2.54mm_Vertical" (id 2) (at 226.695 126.365 0)
+    (property "Footprint" "Connector_PinHeader_2.54mm:PinHeader_1x05_P2.54mm_Vertical" (id 2) (at 226.695 126.365 0)
       (effects (font (size 1.27 1.27)) hide)
     )
@@
     )
     (pin "1")
-  )
-  (symbol (lib_id "Switch:SW_MEC_5G") (at 252.73 132.08 270) (unit 1)
-    (in_bom yes) (on_board yes)
-    (property "Reference" "SW1" (id 0) (at 259.08 131.445 90))
-    (property "Value" "RESET" (id 1) (at 259.08 133.35 90))
-    (property "Footprint" "Button_Switch_SMD:SW_SPST_TL3342" (id 2) (at 257.81 132.08 0)
-      (effects (font (size 1.27 1.27)) hide)
-    )
-    (property "Datasheet" "http://www.apem.com/int/index.php?controller=attachment&id_attachment=488" (id 3) (at 257.81 132.08 0)
-      (effects (font (size 1.27 1.27)) hide)
-    )
-    (pin "1")
-    (pin "3")
-    (pin "2")
-    (pin "4")
   )
   (symbol (lib_id "power:GND") (at 106.68 160.02 0) (unit 1)
@@
     (pin "MP4")
   )
-  (symbol (lib_id "Device:C") (at 63.5 81.915 180) (unit 1)
-    (in_bom yes) (on_board yes)
-    (property "Reference" "C1" (id 0) (at 57.785 81.28 0)
-      (effects (font (size 1.27 1.27)) (justify right))
-    )
-    (property "Value" ".1u" (id 1) (at 57.15 83.185 0)
-      (effects (font (size 1.27 1.27)) (justify right))
-    )
-    (property "Footprint" "Capacitor_SMD:C_0805_2012Metric_Pad1.18x1.45mm_HandSolder" (id 2) (at 62.5348 78.105 0)
+  (symbol (lib_id "Device:C") (at 63.5 81.915 0) (mirror x) (unit 1)
+    (in_bom yes) (on_board yes)
+    (property "Reference" "C1" (id 0) (at 69.215 81.28 0)
+      (effects (font (size 1.27 1.27)) (justify right))
+    )
+    (property "Value" ".1u" (id 1) (at 69.85 83.185 0)
+      (effects (font (size 1.27 1.27)) (justify right))
+    )
+    (property "Footprint" "Capacitor_SMD:C_0805_2012Metric_Pad1.18x1.45mm_HandSolder" (id 2) (at 64.4652 78.105 0)
       (effects (font (size 1.27 1.27)) hide)
     )
@@
     (pin "2")
   )
-  (symbol (lib_id "power:GND") (at 252.73 137.16 0) (unit 1)
-    (in_bom yes) (on_board yes)
-    (property "Reference" "#PWR035" (id 0) (at 252.73 143.51 0)
-      (effects (font (size 1.27 1.27)) hide)
-    )
-    (property "Value" "GND" (id 1) (at 252.73 140.97 0))
-    (property "Footprint" "" (id 2) (at 252.73 137.16 0)
-      (effects (font (size 1.27 1.27)) hide)
-    )
-    (property "Datasheet" "" (id 3) (at 252.73 137.16 0)
+  (symbol (lib_id "Switch:SW_Push") (at 252.73 132.715 270) (unit 1)
+    (in_bom yes) (on_board yes) (fields_autoplaced)
+    (property "Reference" "SW1" (id 0) (at 256.54 131.4449 90)
+      (effects (font (size 1.27 1.27)) (justify left))
+    )
+    (property "Value" "SW_Push" (id 1) (at 256.54 133.9849 90)
+      (effects (font (size 1.27 1.27)) (justify left))
+    )
+    (property "Footprint" "Button_Switch_SMD:SW_SPST_TL3342" (id 2) (at 257.81 132.715 0)
+      (effects (font (size 1.27 1.27)) hide)
+    )
+    (property "Datasheet" "~" (id 3) (at 257.81 132.715 0)
+      (effects (font (size 1.27 1.27)) hide)
+    )
+    (pin "1")
+    (pin "2")
+  )
+  (symbol (lib_id "power:GND") (at 252.73 137.795 0) (unit 1)
+    (in_bom yes) (on_board yes)
+    (property "Reference" "#PWR035" (id 0) (at 252.73 144.145 0)
+      (effects (font (size 1.27 1.27)) hide)
+    )
+    (property "Value" "GND" (id 1) (at 252.73 141.605 0))
+    (property "Footprint" "" (id 2) (at 252.73 137.795 0)
+      (effects (font (size 1.27 1.27)) hide)
+    )
+    (property "Datasheet" "" (id 3) (at 252.73 137.795 0)
       (effects (font (size 1.27 1.27)) hide)
     )
@@
       (reference "#PWR027") (unit 1) (value "VCC") (footprint "")
     )
+    (path "/1e1f074e-e525-4a5f-9c63-f6054393c170"
+      (reference "#PWR028") (unit 1) (value "GND") (footprint "")
+    )
     (path "/3a0f1b58-b58e-4e56-a488-0e8a0136bea6"
-      (reference "#PWR028") (unit 1) (value "VCC") (footprint "")
-    )
-    (path "/1e1f074e-e525-4a5f-9c63-f6054393c170"
-      (reference "#PWR029") (unit 1) (value "GND") (footprint "")
+      (reference "#PWR029") (unit 1) (value "VCC") (footprint "")
     )
     (path "/d3393d47-2d99-4185-baae-1159b56a809b"
@@
     )
     (path "/6075b0ba-f7b4-44be-af4f-53a0ccad088c"
-      (reference "J4") (unit 1) (value "DISPLAY") (footprint "Connector_PinHeader_2.54mm:PinHeader_1x04_P2.54mm_Vertical")
+      (reference "J4") (unit 1) (value "DISPLAY") (footprint "Connector_PinHeader_2.54mm:PinHeader_1x05_P2.54mm_Vertical")
     )
     (path "/014ed757-1d46-4aa5-a651-ebcae908f93b"
@@
       (reference "R12") (unit 1) (value "10k") (footprint "Resistor_SMD:R_0805_2012Metric_Pad1.20x1.40mm_HandSolder")
     )
-    (path "/7b91bbf2-b8d2-4e06-a34c-b820bd7c0e2e"
-      (reference "SW1") (unit 1) (value "RESET") (footprint "Button_Switch_SMD:SW_SPST_TL3342")
+    (path "/f41d233e-5fb2-4e80-a00d-cbb253ff041e"
+      (reference "SW1") (unit 1) (value "SW_Push") (footprint "Button_Switch_SMD:SW_SPST_TL3342")
     )
     (path "/10ee39ec-74d6-47d2-b2b7-0dd8c9f887b7"
