File: builds/3.0/kicad/talking-counter/talking-counter.kicad_sch (KiCad schematic)
At the start: 44 parts, among them IC1 TLV3501AIDR, IC2 LM4862MX_NOPB, J1 Conn_Coaxial, J2 PROG, J3 UJ2-MIBH-G-SMT-TR, SW1 SW_MEC_5E, U2 AP2112K-3.3, U3 AVR64DD32, U4 FT5HV

Commit message: Update talking-counter.kicad_sch
Parts:
- D3: value LED1 -> SIGNAL
- D4: value LED1 -> STATUS
- D6: value LED1 -> POWER
- SW1: value SW_MEC_5E -> SPEAK
- TP1: value SIG_AMP -> AMP_OUT
Changed lines of the file:
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@@
       (effects (font (size 1.27 1.27)))
     )
-    (property "Value" "LED1" (at 119.38 52.07 0)
+    (property "Value" "STATUS" (at 119.38 52.07 0)
       (effects (font (size 1.27 1.27)))
     )
@@
       (effects (font (size 1.27 1.27)))
     )
-    (property "Value" "LED1" (at 119.38 29.21 0)
+    (property "Value" "POWER" (at 119.38 29.21 0)
       (effects (font (size 1.27 1.27)))
     )
@@
       (effects (font (size 1.27 1.27)))
     )
-    (property "Value" "LED1" (at 119.38 40.64 0)
+    (property "Value" "SIGNAL" (at 119.38 40.64 0)
       (effects (font (size 1.27 1.27)))
     )
@@
       (effects (font (size 1.27 1.27)) (justify left))
     )
-    (property "Value" "SW_MEC_5E" (at 257.81 95.25 90)
+    (property "Value" "SPEAK" (at 257.81 95.25 90)
       (effects (font (size 1.27 1.27)) (justify left))
     )
@@
       (effects (font (size 1.27 1.27)) (justify right))
     )
-    (property "Value" "SIG_AMP" (at 151.13 103.632 0)
+    (property "Value" "AMP_OUT" (at 151.13 103.632 0)
       (effects (font (size 1.27 1.27)) (justify right))
     )

Commit message: Update talking-counter.kicad_sch
Parts:
- RV1: footprint Potentiometer_THT:Potentiometer_Alpha_RD901F-40-00D_Single_Vertical -> Potentiometer_THT:Potentiometer_Vishay_T73YP_Vertical
Changed lines of the file:
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@@
       (effects (font (size 1.27 1.27)) (justify right))
     )
-    (property "Footprint" "Potentiometer_THT:Potentiometer_Alpha_RD901F-40-00D_Single_Vertical" (at 36.83 171.45 0)
+    (property "Footprint" "Potentiometer_THT:Potentiometer_Vishay_T73YP_Vertical" (at 36.83 171.45 0)
       (effects (font (size 1.27 1.27)) hide)
     )

Commit message: usbc connector
Parts:
- removed J3: UJ2-MIBH-G-SMT-TR, Connector_USB:USB_Micro-B_Amphenol_10118193-0001LF_Horizontal, symbol library loader:UJ2-MIBH-G-SMT-TR
- added C9: .1u, Capacitor_SMD:C_0805_2012Metric_Pad1.18x1.45mm_HandSolder, symbol Device:C
- added J3: USB_C_Receptacle_PowerOnly_6P, Connector_USB:USB_C_Receptacle_GCT_USB4105-xx-A_16P_TopMnt_Horizontal, symbol Connector:USB_C_Receptacle_PowerOnly_6P
- added R10, R11: 5.1k, Resistor_SMD:R_0805_2012Metric_Pad1.20x1.40mm_HandSolder, symbol Device:R
- added R13: 10k, Resistor_SMD:R_0805_2012Metric_Pad1.20x1.40mm_HandSolder, symbol Device:R
Connections:
- net DAC: now also C9.2, R13.2; no longer U3.16 (PD6)
- net GND: now also C9.1, J3.A12 (GND), J3.B12 (GND), R10.2, R11.2
- net at FB2.1: now also J3.A9 (VBUS), J3.B9 (VBUS)
- new net: J3.B5 (CC2), R10.1
- new net: R13.1, U3.16 (PD6)
- new net: J3.A5 (CC1), R11.1
- no-connect marks 29 -> 23
Other:
- moved on the sheet: C10, C11, D3, D4, D6, FB2, R16, R4, R9, U2

Commit message: create PCB
Parts:
- C1: footprint Jumper:SolderJumper-2_P1.3mm_Open_RoundedPad1.0x1.5mm -> Capacitor_SMD:C_0805_2012Metric_Pad1.18x1.45mm_HandSolder
- J3: footprint Connector_USB:USB_C_Receptacle_GCT_USB4105-xx-A_16P_TopMnt_Horizontal -> Library:USB_C_Receptacle_GCT_USB4105-xx-A_16P_TopMnt_Horizontal
Connections:
- net GND: now also J2.1 (Pin_1); no longer J2.3 (Pin_3)
- net at U3.27 (UPDI): now also J2.3 (Pin_3); no longer J2.1 (Pin_1)
Other:
- moved on the sheet: J2
Changed lines of the file:
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@@
     )
   )
-  (symbol (lib_id "Connector:Conn_01x03_Pin") (at 208.28 35.56 90) (mirror x) (unit 1)
+  (symbol (lib_id "Connector:Conn_01x03_Pin") (at 208.28 35.56 270) (unit 1)
     (in_bom yes) (on_board yes) (dnp no)
     (property "Reference" "J2" (at 208.28 30.48 90)
@@
       (effects (font (size 1.27 1.27)))
     )
-    (property "Footprint" "Connector_USB:USB_C_Receptacle_GCT_USB4105-xx-A_16P_TopMnt_Horizontal" (at 34.29 35.56 0)
+    (property "Footprint" "Library:USB_C_Receptacle_GCT_USB4105-xx-A_16P_TopMnt_Horizontal" (at 34.29 35.56 0)
       (effects (font (size 1.27 1.27)) hide)
     )
@@
       (effects (font (size 1.27 1.27)))
     )
-    (property "Footprint" "Jumper:SolderJumper-2_P1.3mm_Open_RoundedPad1.0x1.5mm" (at 67.945 88.5952 0)
-      (effects (font (size 1.27 1.27)) hide)
-    )
+    (property "Footprint" "Capacitor_SMD:C_0805_2012Metric_Pad1.18x1.45mm_HandSolder" (at 67.945 88.5952 0)
+      (effects (font (size 1.27 1.27)) hide)
+    )
