File: builds/3.0/kicad/talking-counter/talking-counter.kicad_pcb (KiCad board)
At the start: 2 copper layers, 88.9 x 59.7 mm, 52 parts, among them IC1 TLV3501AIDR, IC2 LM4862MX_NOPB, J1 Conn_Coaxial, J2 PROG, J3 USB_C_Receptacle_PowerOnly_6P, SW1 SPEAK, U2 AP2112K-3.3, U3 AVR64DD32, U4 FT5HV

Commit message: update pcb
Routing:
- net Net-(IC2-VO1): track 43.2 -> 38.0 mm
- net Net-(IC2-VO2): track 26.0 -> 23.0 mm
Other:
- board text added: "JLCJLCJLCJLC"
- board text added: "SPEAKER"
Changed lines of the file:
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@@
     (property "ki_keywords" "speaker sound")
     (attr through_hole)
-    (fp_text reference "LS1" (at 0 -0.5 unlocked) (layer "F.SilkS")
+    (fp_text reference "LS1" (at 0 -0.5 unlocked) (layer "F.SilkS") hide
         (effects (font (size 1 1) (thickness 0.1)))
     )
@@
     (effects (font (size 3 3) (thickness 0.375)))
   )
+  (gr_text "SPEAKER" (at 168.91 88.9) (layer "F.SilkS")
+    (effects (font (size 2 2) (thickness 0.15)))
+  )
   (gr_text "STATUS" (at 137.16 133.35) (layer "F.SilkS" knockout)
     (effects (font (size 1.5 1.5) (thickness 0.3) bold))
@@
   (gr_text "Version 3.0 by @swharden" (at 116.332 125.73) (layer "F.SilkS")
     (effects (font (size 1.5 1.5) (thickness 0.1875)) (justify left))
+  )
+  (gr_text "JLCJLCJLCJLC" (at 168.91 97.79) (layer "F.SilkS")
+    (effects (font (size 1 1) (thickness 0.15)) (justify bottom))
   )
   (gr_text "VOLUME" (at 181.356 116.332) (layer "F.SilkS" knockout)
@@
   (segment (start 148.909 114.439) (end 148.909 117.413) (width 0.2) (layer "F.Cu") (net 23))
   (segment (start 162.068 116.84) (end 162.576 116.332) (width 0.25) (layer "F.Cu") (net 23))
+  (segment (start 169.926 92.964) (end 158.004 104.886) (width 0.4) (layer "F.Cu") (net 24))
   (segment (start 157.75 116.332) (end 154.686 116.332) (width 0.4) (layer "F.Cu") (net 24))
   (segment (start 153.859 115.505) (end 153.859 114.439) (width 0.4) (layer "F.Cu") (net 24))
-  (segment (start 158.004 95.996) (end 158.004 116.078) (width 0.4) (layer "F.Cu") (net 24))
-  (segment (start 159.004 94.996) (end 158.004 95.996) (width 0.4) (layer "F.Cu") (net 24))
-  (segment (start 172.212 94.996) (end 159.004 94.996) (width 0.4) (layer "F.Cu") (net 24))
-  (segment (start 174.244 92.964) (end 172.212 94.996) (width 0.4) (layer "F.Cu") (net 24))
+  (segment (start 174.244 92.964) (end 169.926 92.964) (width 0.4) (layer "F.Cu") (net 24))
+  (segment (start 158.004 104.886) (end 158.004 116.078) (width 0.4) (layer "F.Cu") (net 24))
   (segment (start 158.004 116.078) (end 157.75 116.332) (width 0.4) (layer "F.Cu") (net 24))
   (segment (start 154.686 116.332) (end 153.859 115.505) (width 0.4) (layer "F.Cu") (net 24))
-  (segment (start 159.004 92.964) (end 156.718 95.25) (width 0.4) (layer "F.Cu") (net 25))
   (segment (start 156.718 109.474) (end 155.563 110.629) (width 0.4) (layer "F.Cu") (net 25))
-  (segment (start 156.718 95.25) (end 156.718 109.474) (width 0.4) (layer "F.Cu") (net 25))
-  (segment (start 164.084 92.964) (end 159.004 92.964) (width 0.4) (layer "F.Cu") (net 25))
   (segment (start 153.924 110.564) (end 153.859 110.629) (width 0.4) (layer "F.Cu") (net 25))
+  (segment (start 164.084 96.901) (end 156.718 104.267) (width 0.4) (layer "F.Cu") (net 25))
+  (segment (start 156.718 104.267) (end 156.718 109.474) (width 0.4) (layer "F.Cu") (net 25))
+  (segment (start 164.084 92.964) (end 164.084 96.901) (width 0.4) (layer "F.Cu") (net 25))
   (segment (start 155.563 110.629) (end 153.859 110.629) (width 0.4) (layer "F.Cu") (net 25))
   (segment (start 109.22 102.87) (end 109.22 95.25) (width 0.4) (layer "F.Cu") (net 26))
